File: KICAD/jrNIC_v05/jrNIC_v05.kicad_sch (KiCad schematic)
At the start: 6 parts, among them U1 74LS04, U2 74LS08, U3 74LS00, U4 74LS138, U5 74LS138

Commit message: Added RESET latch
Parts:
- removed U3: 74LS00, symbol 74xx:74LS00
- removed U4, U5: 74LS138, symbol 74xx:74LS138
- added C1, C2, C3, C4, C5: 47pF, Capacitor_THT:CP_Radial_Tantal_D5.0mm_P2.50mm, symbol Device:C
- added C6, C8: 10uF, Capacitor_THT:CP_Radial_D5.0mm_P2.50mm, symbol Device:C
- added C7: 100nF, Capacitor_THT:CP_Radial_D5.0mm_P2.50mm, symbol Device:C
- added D1, D2: LED, LED_THT:LED_D3.0mm, symbol Device:LED
- added J2: ~, PCjr_PROTO_RAM_CART_footprint_lib:Olimex_ENC28J60-H, symbol PCjr_PROTO_RAM_CART_symbol_lib:Ethernet_DevBoard
- added J3, J4: Conn_02x03_Odd_Even, Connector_PinHeader_2.54mm:PinHeader_2x03_P2.54mm_Vertical, symbol Connector_Generic:Conn_02x03_Odd_Even
- added J5: Conn_02x05_Odd_Even, Connector_PinHeader_2.54mm:PinHeader_2x05_P2.54mm_Vertical, symbol Connector_Generic:Conn_02x05_Odd_Even
- added R1, R2: 120, Resistor_THT:R_Axial_DIN0204_L3.6mm_D1.6mm_P2.54mm_Vertical, symbol Device:R
- added U3: 74LS138, Package_DIP:DIP-16_W7.62mm_LongPads, symbol 74xx:74LS138
- added U4: 74LS00, Package_DIP:DIP-14_W7.62mm_LongPads, symbol 74xx:74LS00
- added U5: 74LS244, Package_DIP:DIP-20_W7.62mm_LongPads, symbol 74xx:74LS244
- added U6: ~, Package_TO_SOT_THT:TO-220-3_Vertical, symbol PCjr_PROTO_RAM_CART_symbol_lib:LD1117V33
- U1, U2: footprint (none) -> Package_DIP:DIP-14_W7.62mm_LongPads
Connections:
- net 5V is gone; now on net +5V: J1.A14 (5V), J1.B1 (5V), J1.B15 (5V)
- net A0: now also U3.1 (A0)
- net A1: now also U3.2 (A1)
- net A2: now also U3.3 (A2)
- net A9: now also U2.2; no longer U2.1
- net D0: now also U5.18 (O0a)
- net D7: now also J2.2 (COPI), J5.3 (Pin_3)
- net GND: now also U1.7 (GND), U2.7 (GND), C1.2, C2.2, C3.2, C4.2, C5.2, C6.2, C7.2, C8.2, J2.9 (GND), J3.2 (Pin_2), J3.4 (Pin_4), J3.6 (Pin_6), J4.2 (Pin_2), J4.4 (Pin_4), J4.6 (Pin_6), J5.4 (Pin_4), R1.2, R2.2, U3.4 (E1), U3.5 (E2), U3.8 (GND), U4.10, U4.12, U4.13, U4.7 (GND), U4.9, U5.10 (GND), U5.11 (I0b), U5.13 (I1b), U5.15 (I2b), U5.17 (I3b), U5.4 (I1a), U5.6 (I2a), U5.8 (I3a), U6.1 (GND)
- net IOR: now also U1.6, U2.10; no longer U1.4, U2.5
- net IOW: now also U1.4, U2.5; no longer U1.6, U2.10
- net MODEM_CS: now also U2.1; no longer U2.2
- net MODEM_INT: now also U1.12
- net READ_SELECT: now also U1.9, U2.8; no longer U2.6
- net WRITE_SELECT: now also U2.6, U3.6 (E3); no longer U2.8
- net ~{IOR}: now also U1.5; no longer U1.3
- net ~{IOW}: now also U1.3; no longer U1.5
- net ~{RESET}: now also U2.13
- net +12V: now reaches J1.A15 (12V)
- net ~{LATCH_R_COMBINED}: now reaches U2.11
- net ~{LATCH_R_COMBINED}: now also U4.5
- net ~{LATCH_R}: now reaches U2.12
- net ~{LATCH_R}: now also U3.9 (O6)
- net ~{READ_SELECT}: now reaches U1.8
- net ~{READ_SELECT}: now also U5.1 (OEa), U5.19 (OEb)
- net +5V: now reaches U2.14 (VCC)
- net +5V: now also U1.14 (VCC), C1.1, C2.1, C3.1, C4.1, C5.1, C6.1, C7.1, D2.2 (A), J3.1 (Pin_1), J3.3 (Pin_3), J3.5 (Pin_5), U3.16 (VCC), U4.14 (VCC), U5.20 (VCC), U6.3 (VIN)
- net CLK: now reaches U1.10
- net CLK: now also J2.1 (CLK), J5.1 (Pin_1)
- net ~{CLK}: now reaches U1.11
- net ~{CLK}: now also U3.10 (O5)
- net ~{ETH_INT}: now reaches U1.13
- net ~{ETH_INT}: now also J2.5 (~{INT}), J5.9 (Pin_9)
- net D1: no longer names the net of J1.A9 (D1)
- net D2: no longer names the net of J1.A7 (D2)
- net D3: no longer names the net of J1.A6 (D3)
- net D4: no longer names the net of J1.A5 (D4)
- net D5: no longer names the net of J1.A3 (D5)
- net D6: no longer names the net of J1.A2 (D6)
- net JRNIC_SELECT renamed MODEM_PORT
- new net: D2.1 (K), R2.1
- new net: D1.1 (K), R1.1
- new net +3.3V: C8.1, J2.10 (3.3V), J2.8 (~{ETH_RESET}), J4.1 (Pin_1), J4.3 (Pin_3), J4.5 (Pin_5), J5.2 (Pin_2), J5.6 (Pin_6), U6.2 (VOUT)
- new net CIPO: J2.3 (CIPO), J5.5 (Pin_5), U5.2 (I0a)
- new net CLK_OUTx: J2.6 (CLK_OUT), J5.10 (Pin_10)
- new net ETH_CS: D1.2 (A), U4.3, U4.4
- new net ~{ETH_CS}: J2.7 (~{CS}), J5.8 (Pin_8), U4.2, U4.6
- new net ~{LATCH_S}: U3.7 (O7), U4.1
- no-connect marks 4 -> 25
Other:
- note added: "+3.3V Debug Header"
- note added: "+5V Debug Header"
- note added: "3.3V Regulator and caps"
- note added: "Eth Debug Header"
- note added: "Ethernet Controller Dev Board"
- note added: "IC Power"
- note added: "Indicator LEDs"
- note added: "Logical Power"
- note added: "PCjr Modem Slot"
- note added: "PCjr Signaling Technical Reference 2-29 I/O Channel I/O Map Table - 98 7654 3210 - 00 1111 Xaaa - Port 0F8-0FF (Diskette) [For Reference] - 10 1111 1aaa - Port 2F8-2FF (Serial Port) [For Reference] - 11 1111 1aaa - Port 3F8-3FF (Modem) Technical Reference 3-70 Internal Modem - IQR4 (Positive-Active) Technical Reference 3-72 Internal Modem ~{MODEM_CS}/~{DISKETTE_CS} is asserted low for both Modem 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"
- note added: "Power bypass capacitors"
- note added: "Power-up Force Latch"
- note added: "Prototype 1 - Raw bit-bang, manually shift bits together on PCjr side -Goals: 1.) Read/Write data successfully from ethernet controller - works 2.) Get interrupt to trigger - works 3.) Implement mimimal packet driver - in progress Most of the focus will be here, will keep this design unless it ends up breaking mTCP Possible future protoypes: Prototype 2 - Add Shift register (may or may not need 3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"
- note added: "SR Latch ~{S}~{R} E~{E} 10 01 01 10 11 no change 00 invalid"
- note added: "SR-Latch"
- note added: "Spare"
- note added: "TODO DONE-Use reset to also control S/R latch Reset -Shift register -Auto Shift Register -Find a level shifter -Use reset + level shifter to control ethernet controller reset as well -Find a 3.3V Regulator - currently "abuses" the tolerances of the 74LS chips -Potentially re-implement the previously shelved shift register logic -Add IC caps and board bulk cap"
- note removed: "NOR 001 010 100 110"
- note removed: "PCjr Modem Port"
- note removed: "PCjr Signaling Technical Reference 2-29 I/O Channel I/O Map Table - 98 7654 3210 - 00 1111 Xaaa - Port 0F8-0FF (Diskette) [For Reference] - 10 1111 1aaa - Port 2F8-2FF (Serial Port) [For Reference] - 11 1111 1aaa - Port 3F8-3FF (Modem) Technical Reference 3-70 Internal Modem - IRQ4 (Positive-Active) Technical Reference 3-72 Internal Modem ~{MODEM_CS}/~{DISKETTE_CS} is asserted low for both Modem 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"
- note removed: "SR Latch (NAND) ~{S}~{R} E~{E} 10 01 01 10 11 no change 00 invalid"
- note removed: "SR Latch (NOR) ~{S}~{R} E~{E} 10 01 01 10 11 no change 00 invalid"
